File: output/modular-output.sch (KiCad schematic (older format))
At the start: 15 parts, among them J1 Conn_02x05_Odd_Even, J2 Conn_01x02, J3 Conn_01x05, J4 Audio-Jack-3, SW1 SW_SPDT, U1 TL072

Commit message: output module schema again
Parts:
- added SW?: SW_SPDT, symbol SW_SPDT
Connections:
- net at C2.1, J3.3 (Pin_3), R4.1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: now also SW?.1 (A); no longer J4.1
- net at C1.1, J3.1 (Pin_1), J4.2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: now also SW?.3 (C)
- net at C1.2, R3.2, U1.2 (-): now also SW1.1 (A); no longer R1.1
- net at R2.2, RV1.5: no longer SW1.1 (A)
- net at SW1.2 (B): now also R1.1; no longer R1.2
- net at SW1.3 (C): no longer RV1.2
- new net: J4.1, SW?.2 (B)
- new net: R1.2, RV1.2
Other:
- moved on the sheet: R1, R2, SW1
Changed lines of the file:
@@
 L SW_SPDT SW1
 U 1 1 5C071DC8
-P 3850 3250
-F 0 "SW1" H 3850 3420 50  0000 C CNN
-F 1 "SW_SPDT" H 3850 3050 50  0000 C CNN
-F 2 "" H 3850 3250 50  0001 C CNN
-F 3 "" H 3850 3250 50  0001 C CNN
-	1    3850 3250
-	-1   0    0    1
+P 4150 3350
+F 0 "SW1" H 4150 3520 50  0000 C CNN
+F 1 "SW_SPDT" H 4150 3150 50  0000 C CNN
+F 2 "" H 4150 3350 50  0001 C CNN
+F 3 "" H 4150 3350 50  0001 C CNN
+	1    4150 3350
+	1    0    0    -1
 $EndComp
 $Comp
@@
 L R R2
 U 1 1 5C072FFD
-P 4300 3650
-F 0 "R2" V 4380 3650 50  0000 C CNN
-F 1 "100k" V 4300 3650 50  0000 C CNN
-F 2 "" V 4230 3650 50  0001 C CNN
-F 3 "" H 4300 3650 50  0001 C CNN
-	1    4300 3650
+P 3600 3650
+F 0 "R2" V 3680 3650 50  0000 C CNN
+F 1 "100k" V 3600 3650 50  0000 C CNN
+F 2 "" V 3530 3650 50  0001 C CNN
+F 3 "" H 3600 3650 50  0001 C CNN
+	1    3600 3650
 	0    1    1    0
 $EndComp
@@
 L R R1
 U 1 1 5C07307A
-P 4300 3150
-F 0 "R1" V 4380 3150 50  0000 C CNN
-F 1 "100k" V 4300 3150 50  0000 C CNN
-F 2 "" V 4230 3150 50  0001 C CNN
-F 3 "" H 4300 3150 50  0001 C CNN
-	1    4300 3150
+P 3600 3150
+F 0 "R1" V 3680 3150 50  0000 C CNN
+F 1 "100k" V 3600 3150 50  0000 C CNN
+F 2 "" V 3530 3150 50  0001 C CNN
+F 3 "" H 3600 3150 50  0001 C CNN
+	1    3600 3150
 	0    1    1    0
 $EndComp
@@
 $EndComp
 Wire Wire Line
-	4450 3650 4450 4450
+	4450 3450 4450 4450
 Wire Wire Line
 	4450 4450 4850 4450
@@
 	5150 3850 5450 3850
 Connection ~ 5450 3850
-Wire Wire Line
-	5450 4550 6400 4550
 $Comp
 L -VDC #PWR04
@@
 	4850 2700 4450 2700
 Wire Wire Line
-	4450 2700 4450 3150
+	4450 2700 4450 3250
 $Comp
 L R R3
@@
 to headphone amp submodule
 Wire Wire Line
-	6400 4550 6400 3700
-Wire Wire Line
 	6400 2800 6400 3600
 $Comp
@@
 	5750 5300 5950 5300
 Wire Wire Line
-	3450 3150 3650 3150
-Wire Wire Line
-	4050 3250 4100 3250
-Wire Wire Line
-	4100 3250 4100 3150
-Wire Wire Line
-	4100 3150 4150 3150
-Wire Wire Line
-	3450 3650 4150 3650
-Wire Wire Line
-	3650 3350 3650 3650
-Connection ~ 3650 3650
+	3750 3150 3950 3150
+Wire Wire Line
+	4450 3250 4350 3250
+Wire Wire Line
+	3750 3650 4450 3650
 Wire Wire Line
 	3250 3000 2750 3000
@@
 Wire Wire Line
 	2750 3500 3250 3500
+Wire Wire Line
+	3950 3150 3950 3350
+Wire Wire Line
+	4400 3450 4450 3450
+Connection ~ 4450 3650
+$Comp
+L SW_SPDT SW?
+U 1 1 5C5D5C7E
+P 6200 4150
+F 0 "SW?" V 6200 4320 50  0000 C CNN
+F 1 "SW_SPDT" H 6200 3950 50  0000 C CNN
+F 2 "" H 6200 4150 50  0001 C CNN
+F 3 "" H 6200 4150 50  0001 C CNN
+	1    6200 4150
+	-1   0    0    1
+$EndComp
+Wire Wire Line
+	6400 4150 6400 3700
+Wire Wire Line
+	6000 4050 5950 4050
+Connection ~ 5950 4050
+Wire Wire Line
+	6000 4250 6000 4550
+Wire Wire Line
+	6000 4550 5450 4550
 $EndSCHEMATC

Commit message: output: dc block
Parts:
- added C3, C4: 820n, symbol C
- gave numbers to parts that had none: 1
Connections:
- net at C2.2, R2.1, R4.2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: now also SW1.3 (C)
- net at J2.1 (Pin_1): now also C4.2; no longer RV1.4
- net at J2.2 (Pin_2): now also C3.2; no longer RV1.1
- new net: C3.1, RV1.1
- new net: C4.1, RV1.4
Other:
- moved on the sheet: R1, R2

Commit message: output: zener diodes
Parts:
- added D1, D2, D3, D4: D_Zener, symbol D_Zener
- added R5, R6: 1k, symbol R
Connections:
- net GND: now also D1.1 (K), D4.1 (K)
- net at RV1.2: now also R5.2; no longer R1.2
- net at RV1.5: now also R6.2; no longer R2.2
- new net: D3.1 (K), R2.2, R6.1
- new net: D2.1 (K), R1.2, R5.1
- new net: D1.2 (A), D2.2 (A)
- new net: D3.2 (A), D4.2 (A)
Other:
- moved on the sheet: C3, C4, J2, RV1

Commit message: output: tweaks and fixes
Parts:
- removed SW1, SW2: SW_SPDT, symbol SW_SPDT
- added SW1: SW_DPDT_x2, symbol SW_DPDT_x2
Connections:
- net at J4.1: now also C2.1, J3.3 (Pin_3), R4.1, U1.7, SW1.6 (C)
- net at C1.1, R3.1, U1.1: now also SW1.4 (A); no longer J3.1 (Pin_1), J4.2
- net at C2.2, R2.1, R4.2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: now also SW1.3 (C)
- net at C1.2, R3.2, U1.2 (-): now also SW1.1 (A)
- net at R1.1: now also SW1.2 (B)
- new net: J3.1 (Pin_1), J4.2, SW1.5 (B)
Other:
- moved on the sheet: J3, J4, R3, R4
Changed lines of the file:
@@
 L Audio-Jack-3 J4
 U 1 1 5C071850
-P 6600 3700
-F 0 "J4" H 6550 3875 50  0000 C CNN
-F 1 "Audio-Jack-3" H 6700 3630 50  0000 C CNN
-F 2 "" H 6850 3800 50  0001 C CNN
-F 3 "" H 6850 3800 50  0001 C CNN
-	1    6600 3700
+P 6800 3500
+F 0 "J4" H 6750 3675 50  0000 C CNN
+F 1 "Audio-Jack-3" H 6900 3430 50  0000 C CNN
+F 2 "" H 7050 3600 50  0001 C CNN
+F 3 "" H 7050 3600 50  0001 C CNN
+	1    6800 3500
 	-1   0    0    -1
 $EndComp
@@
 $EndComp
 $Comp
-L SW_SPDT SW1
-U 1 1 5C071DC8
-P 4150 3350
-F 0 "SW1" H 4150 3520 50  0000 C CNN
-F 1 "SW_SPDT" H 4150 3150 50  0000 C CNN
-F 2 "" H 4150 3350 50  0001 C CNN
-F 3 "" H 4150 3350 50  0001 C CNN
-	1    4150 3350
-	1    0    0    -1
-$EndComp
-$Comp
 L POT_Dual RV1
 U 1 1 5C072241
@@
 L R R4
 U 1 1 5C0732C3
-P 5000 3850
-F 0 "R4" V 5080 3850 50  0000 C CNN
-F 1 "10k" V 5000 3850 50  0000 C CNN
-F 2 "" V 4930 3850 50  0001 C CNN
-F 3 "" H 5000 3850 50  0001 C CNN
-	1    5000 3850
+P 5300 3850
+F 0 "R4" V 5380 3850 50  0000 C CNN
+F 1 "10k" V 5300 3850 50  0000 C CNN
+F 2 "" V 5230 3850 50  0001 C CNN
+F 3 "" H 5300 3850 50  0001 C CNN
+	1    5300 3850
 	0    1    1    0
 $EndComp
@@
 L R R3
 U 1 1 5C074018
-P 5000 2100
-F 0 "R3" V 5080 2100 50  0000 C CNN
-F 1 "10k" V 5000 2100 50  0000 C CNN
-F 2 "" V 4930 2100 50  0001 C CNN
-F 3 "" H 5000 2100 50  0001 C CNN
-	1    5000 2100
+P 5300 2100
+F 0 "R3" V 5380 2100 50  0000 C CNN
+F 1 "10k" V 5300 2100 50  0000 C CNN
+F 2 "" V 5230 2100 50  0001 C CNN
+F 3 "" H 5300 2100 50  0001 C CNN
+	1    5300 2100
 	0    1    1    0
 $EndComp
@@
 L GND #PWR012
 U 1 1 5C074CC4
-P 5600 5100
-F 0 "#PWR012" H 5600 4850 50  0001 C CNN
-F 1 "GND" H 5600 4950 50  0000 C CNN
-F 2 "" H 5600 5100 50  0001 C CNN
-F 3 "" H 5600 5100 50  0001 C CNN
-	1    5600 5100
-	1    0    0    -1
-$EndComp
-Text Notes 6300 5200 0    60   ~ 0
+P 6200 5100
+F 0 "#PWR012" H 6200 4850 50  0001 C CNN
+F 1 "GND" H 6200 4950 50  0000 C CNN
+F 2 "" H 6200 5100 50  0001 C CNN
+F 3 "" H 6200 5100 50  0001 C CNN
+	1    6200 5100
+	1    0    0    -1
+$EndComp
+Text Notes 6900 5200 0    60   ~ 0
 to headphone amp submodule
 $Comp
 L GND #PWR013
 U 1 1 5C074F87
-P 6800 3800
-F 0 "#PWR013" H 6800 3550 50  0001 C CNN
-F 1 "GND" H 6800 3650 50  0000 C CNN
-F 2 "" H 6800 3800 50  0001 C CNN
-F 3 "" H 6800 3800 50  0001 C CNN
-	1    6800 3800
+P 7000 3600
+F 0 "#PWR013" H 7000 3350 50  0001 C CNN
+F 1 "GND" H 7000 3450 50  0000 C CNN
+F 2 "" H 7000 3600 50  0001 C CNN
+F 3 "" H 7000 3600 50  0001 C CNN
+	1    7000 3600
 	1    0    0    -1
 $EndComp
@@
 L Conn_01x05 J3
 U 1 1 5C076332
-P 6150 5200
-F 0 "J3" H 6150 5500 50  0000 C CNN
-F 1 "Conn_01x05" H 6150 4900 50  0000 C CNN
-F 2 "" H 6150 5200 50  0001 C CNN
-F 3 "" H 6150 5200 50  0001 C CNN
-	1    6150 5200
+P 6750 5200
+F 0 "J3" H 6750 5500 50  0000 C CNN
+F 1 "Conn_01x05" H 6750 4900 50  0000 C CNN
+F 2 "" H 6750 5200 50  0001 C CNN
+F 3 "" H 6750 5200 50  0001 C CNN
+	1    6750 5200
 	1    0    0    -1
 $EndComp
@@
 L -VDC #PWR020
 U 1 1 5C076385
-P 5950 5400
-F 0 "#PWR020" H 5950 5300 50  0001 C CNN
-F 1 "-VDC" H 5950 5650 50  0000 C CNN
-F 2 "" H 5950 5400 50  0001 C CNN
-F 3 "" H 5950 5400 50  0001 C CNN
-	1    5950 5400
+P 6550 5400
+F 0 "#PWR020" H 6550 5300 50  0001 C CNN
+F 1 "-VDC" H 6550 5650 50  0000 C CNN
+F 2 "" H 6550 5400 50  0001 C CNN
+F 3 "" H 6550 5400 50  0001 C CNN
+	1    6550 5400
 	-1   0    0    1
 $EndComp
@@
 L +VDC #PWR021
 U 1 1 5C0763C9
-P 5750 5300
-F 0 "#PWR021" H 5750 5200 50  0001 C CNN
-F 1 "+VDC" H 5750 5550 50  0000 C CNN
-F 2 "" H 5750 5300 50  0001 C CNN
-F 3 "" H 5750 5300 50  0001 C CNN
-	1    5750 5300
-	-1   0    0    1
-$EndComp
-$Comp
-L SW_SPDT SW2
-U 1 1 5C5D5C7E
-P 6200 4150
-F 0 "SW2" V 6200 4320 50  0000 C CNN
-F 1 "SW_SPDT" H 6200 3950 50  0000 C CNN
-F 2 "" H 6200 4150 50  0001 C CNN
-F 3 "" H 6200 4150 50  0001 C CNN
-	1    6200 4150
+P 6350 5300
+F 0 "#PWR021" H 6350 5200 50  0001 C CNN
+F 1 "+VDC" H 6350 5550 50  0000 C CNN
+F 2 "" H 6350 5300 50  0001 C CNN
+F 3 "" H 6350 5300 50  0001 C CNN
+	1    6350 5300
 	-1   0    0    1
 $EndComp
@@
 Wire Wire Line
 	5450 3650 5150 3650
-Wire Wire Line
-	5150 3850 5450 3850
 Connection ~ 5450 3850
 Wire Wire Line
@@
 Wire Wire Line
 	5450 1900 5150 1900
-Wire Wire Line
-	5150 2100 5450 2100
 Connection ~ 5450 2100
 Wire Wire Line
-	5450 2800 6400 2800
-Wire Wire Line
-	5950 5000 5950 2800
-Connection ~ 5950 2800
-Wire Wire Line
-	5950 5200 5800 5200
-Wire Wire Line
-	5800 5200 5800 4550
-Connection ~ 5800 4550
-Wire Wire Line
-	5950 5100 5600 5100
-Wire Wire Line
-	6400 2800 6400 3600
-Wire Wire Line
-	5750 5300 5950 5300
+	6350 5200 6550 5200
+Wire Wire Line
+	6550 5100 6200 5100
+Wire Wire Line
+	6350 5300 6550 5300
 Wire Wire Line
 	4450 3250 4350 3250
@@
 	4350 3450 4450 3450
 Connection ~ 4450 3650
-Wire Wire Line
-	6400 4150 6400 3700
-Wire Wire Line
-	6000 4050 5950 4050
-Connection ~ 5950 4050
-Wire Wire Line
-	6000 4250 6000 4550
-Wire Wire Line
-	6000 4550 5450 4550
 Wire Wire Line
 	2450 3000 2650 3000
@@
 Connection ~ 3500 3950
 Connection ~ 3500 2850
+$Comp
+L SW_DPDT_x2 SW1
+U 1 1 5C5DAA8E
+P 4150 3350
+F 0 "SW1" H 4150 3520 50  0000 C CNN
+F 1 "SW_DPDT_x2" H 4150 3150 50  0000 C CNN
+F 2 "" H 4150 3350 50  0001 C CNN
+F 3 "" H 4150 3350 50  0001 C CNN
+	1    4150 3350
+	1    0    0    -1
+$EndComp
+$Comp
+L SW_DPDT_x2 SW1
+U 2 1 5C5DAB25
+P 6150 3400
+F 0 "SW1" H 6150 3570 50  0000 C CNN
+F 1 "SW_DPDT_x2" H 6150 3200 50  0000 C CNN
+F 2 "" H 6150 3400 50  0001 C CNN
+F 3 "" H 6150 3400 50  0001 C CNN
+	2    6150 3400
+	-1   0    0    -1
+$EndComp
+Wire Wire Line
+	5450 4550 6600 4550
+Wire Wire Line
+	6600 4550 6600 3500
+Wire Wire Line
+	6600 3400 6350 3400
+Wire Wire Line
+	5950 3300 5950 2800
+Wire Wire Line
+	5950 2800 5450 2800
+Wire Wire Line
+	5950 3500 5950 4550
+Connection ~ 5950 4550
+Wire Wire Line
+	6350 5200 6350 4550
+Connection ~ 6350 4550
+Wire Wire Line
+	6550 5000 6450 5000
+Wire Wire Line
+	6450 5000 6450 3400
+Connection ~ 6450 3400
+Connection ~ 5450 4550
+Connection ~ 4850 4450
+Connection ~ 4850 2700
+Connection ~ 5450 2800
+Wire Wire Line
+	5150 2100 4850 2100
+Wire Wire Line
+	5150 3850 4850 3850
 $EndSCHEMATC

Commit message: output: some changes
Parts:
- removed J3: Conn_01x05, symbol Conn_01x05
- removed J4: Audio-Jack-3, symbol Audio-Jack-3
- added J? (x2): Conn_02x03_Odd_Even, symbol Conn_02x03_Odd_Even
Connections:
- net GND: now also J?.5 (Pin_5), J?.5 (Pin_5), J?.6 (Pin_6), J?.6 (Pin_6)
- net at C2.1, R4.1, SW1.6 (C)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: now also J?.3 (Pin_3), J?.3 (Pin_3), J?.4 (Pin_4), J?.4 (Pin_4)
- net at SW1.5 (B): now also J?.1 (Pin_1), J?.1 (Pin_1), J?.2 (Pin_2), J?.2 (Pin_2)
Changed lines of the file:
@@
-$EndComp
-$Comp
-L Audio-Jack-3 J4
-U 1 1 5C071850
-P 6800 3500
-F 0 "J4" H 6750 3675 50  0000 C CNN
-F 1 "Audio-Jack-3" H 6900 3430 50  0000 C CNN
-F 2 "" H 7050 3600 50  0001 C CNN
-F 3 "" H 7050 3600 50  0001 C CNN
-	1    6800 3500
-	-1   0    0    -1
 $EndComp
 $Comp
@@
 	1    0    0    -1
 $EndComp
-$Comp
-L GND #PWR012
-U 1 1 5C074CC4
-P 6200 5100
-F 0 "#PWR012" H 6200 4850 50  0001 C CNN
-F 1 "GND" H 6200 4950 50  0000 C CNN
-F 2 "" H 6200 5100 50  0001 C CNN
-F 3 "" H 6200 5100 50  0001 C CNN
-	1    6200 5100
-	1    0    0    -1
-$EndComp
 Text Notes 6900 5200 0    60   ~ 0
 to headphone amp submodule
-$Comp
-L GND #PWR013
-U 1 1 5C074F87
-P 7000 3600
-F 0 "#PWR013" H 7000 3350 50  0001 C CNN
-F 1 "GND" H 7000 3450 50  0000 C CNN
-F 2 "" H 7000 3600 50  0001 C CNN
-F 3 "" H 7000 3600 50  0001 C CNN
-	1    7000 3600
-	1    0    0    -1
-$EndComp
 NoConn ~ 2350 5000
 NoConn ~ 2850 5000
@@
 $EndComp
 $Comp
-L Conn_01x05 J3
-U 1 1 5C076332
-P 6750 5200
-F 0 "J3" H 6750 5500 50  0000 C CNN
-F 1 "Conn_01x05" H 6750 4900 50  0000 C CNN
-F 2 "" H 6750 5200 50  0001 C CNN
-F 3 "" H 6750 5200 50  0001 C CNN
-	1    6750 5200
-	1    0    0    -1
-$EndComp
-$Comp
-L -VDC #PWR020
-U 1 1 5C076385
-P 6550 5400
-F 0 "#PWR020" H 6550 5300 50  0001 C CNN
-F 1 "-VDC" H 6550 5650 50  0000 C CNN
-F 2 "" H 6550 5400 50  0001 C CNN
-F 3 "" H 6550 5400 50  0001 C CNN
-	1    6550 5400
-	-1   0    0    1
-$EndComp
-$Comp
-L +VDC #PWR021
-U 1 1 5C0763C9
-P 6350 5300
-F 0 "#PWR021" H 6350 5200 50  0001 C CNN
-F 1 "+VDC" H 6350 5550 50  0000 C CNN
-F 2 "" H 6350 5300 50  0001 C CNN
-F 3 "" H 6350 5300 50  0001 C CNN
-	1    6350 5300
-	-1   0    0    1
-$EndComp
-$Comp
 L C C3
 U 1 1 5C5D60A8
@@
 Connection ~ 5450 2100
 Wire Wire Line
-	6350 5200 6550 5200
-Wire Wire Line
-	6550 5100 6200 5100
-Wire Wire Line
-	6350 5300 6550 5300
-Wire Wire Line
 	4450 3250 4350 3250
 Wire Wire Line
@@
 	3350 3150 3650 3150
 Wire Wire Line
-	3650 3650 3350 3650
+	3350 3650 3650 3650
 $Comp
 L D_Zener D2
@@
 $EndComp
 Wire Wire Line
-	5450 4550 6600 4550
-Wire Wire Line
-	6600 4550 6600 3500
-Wire Wire Line
-	6600 3400 6350 3400
+	5450 4550 6400 4550
+Wire Wire Line
+	6350 3400 7950 3400
 Wire Wire Line
 	5950 3300 5950 2800
@@
 	5950 3500 5950 4550
 Connection ~ 5950 4550
-Wire Wire Line
-	6350 5200 6350 4550
-Connection ~ 6350 4550
-Wire Wire Line
-	6550 5000 6450 5000
-Wire Wire Line
-	6450 5000 6450 3400
-Connection ~ 6450 3400
 Connection ~ 5450 4550
 Connection ~ 4850 4450
@@
 Wire Wire Line
 	5150 3850 4850 3850
+$Comp
+L Conn_02x03_Odd_Even J?
+U 1 1 5C61AB41
+P 6800 3500
+F 0 "J?" H 6850 3700 50  0000 C CNN
+F 1 "Conn_02x03_Odd_Even" H 6850 3300 50  0000 C CNN
+F 2 "" H 6800 3500 50  0001 C CNN
+F 3 "" H 6800 3500 50  0001 C CNN
+	1    6800 3500
+	1    0    0    -1
+$EndComp
+$Comp
+L Conn_02x03_Odd_Even J?
+U 1 1 5C61AC08
+P 7650 3500
+F 0 "J?" H 7700 3700 50  0000 C CNN
+F 1 "Conn_02x03_Odd_Even" H 7700 3300 50  0000 C CNN
+F 2 "" H 7650 3500 50  0001 C CNN
+F 3 "" H 7650 3500 50  0001 C CNN
+	1    7650 3500
+	1    0    0    -1
+$EndComp
+Wire Wire Line
+	6400 3500 7950 3500
+Wire Wire Line
+	6400 4550 6400 3500
+Connection ~ 6600 3400
+Connection ~ 6600 3500
+Wire Wire Line
+	6600 3600 8200 3600
+Connection ~ 7100 3400
+Connection ~ 7450 3400
+Connection ~ 7450 3500
+Connection ~ 7100 3500
+Connection ~ 7100 3600
+Connection ~ 7450 3600
+$Comp
+L GND #PWR?
+U 1 1 5C61AFE2
+P 8200 3600
+F 0 "#PWR?" H 8200 3350 50  0001 C CNN
+F 1 "GND" H 8200 3450 50  0000 C CNN
+F 2 "" H 8200 3600 50  0001 C CNN
+F 3 "" H 8200 3600 50  0001 C CNN
+	1    8200 3600
+	1    0    0    -1
+$EndComp
+Connection ~ 7950 3600
 $EndSCHEMATC
